Commit message: Adding obstacles (ground urdf), tuning the task gains, adding some push experiments

File: project/urdf/obstacles.urdf (robot description, URDF)
Before this commit: robot ground_skeleton, 7 links, 6 joints
Links:
- removed link ground_link
- link s_0: geometry collision box size=0.045 0.3 0.0; visual box size=0.045 0.3 0.015
- link s_1: geometry collision box size=0.25 0.6 0.015; visual box size=0.25 0.6 0.015
- link s_2: geometry collision box size=0.25 0.6 0.015; visual box size=0.25 0.6 0.015
- link s_3: geometry collision box size=0.25 0.6 0.015; visual box size=0.25 0.6 0.015
- link s_4: geometry collision box size=0.25 0.6 0.015; visual box size=0.25 0.6 0.015
Joints:
- removed joint ground_joint
- joint joint_s_0_s_1: origin xyz=0.6 0.3 0 rpy=0 0 0 -> xyz=0.95 0 0 rpy=0 0 0
- joint joint_s_1_s_2: origin xyz=0.6 -0.3 0 rpy=0 0 0 -> xyz=0.95 0 0 rpy=0 0 0
- joint joint_s_2_s_3: origin xyz=0.6 0.3 0 rpy=0 0 0 -> xyz=0.95 0 0 rpy=0 0 0
- joint joint_s_3_s_4: origin xyz=0.6 -0.3 0.0 rpy=0 0 0 -> xyz=0.95 0 0.0 rpy=0 0 0
- joint joint_world_s_0: origin xyz=0.6 -0.15 0.5 rpy=0 0 0 -> xyz=0.92 -0.15 0 rpy=0 0 0; parent ground_link -> world

File: project/urdf/stairs.urdf (robot description, URDF)
Before this commit: robot ground_skeleton, 7 links, 6 joints
Links:
- removed link ground_link
- link s_0: geometry collision box size=0.6 0.3 0.025; visual box size=0.6 0.3 0.025
- link s_1: geometry collision box size=0.6 0.3 0.025; visual box size=0.6 0.3 0.025
- link s_2: geometry collision box size=0.6 0.3 0.025; visual box size=0.6 0.3 0.025
- link s_3: geometry collision box size=0.6 0.3 0.025; visual box size=0.6 0.3 0.025
- link s_4: geometry collision box size=0.6 0.3 0.025; visual box size=0.6 0.3 0.025
Joints:
- removed joint ground_joint
- joint joint_s_0_s_1: origin xyz=0.6 0.3 0 rpy=0 0 0 -> xyz=0.4 0 0.025 rpy=0 0 0
- joint joint_s_1_s_2: origin xyz=0.6 -0.3 0 rpy=0 0 0 -> xyz=0.4 0 0.025 rpy=0 0 0
- joint joint_s_2_s_3: origin xyz=0.6 0.3 0 rpy=0 0 0 -> xyz=0.4 0 0.025 rpy=0 0 0
- joint joint_s_3_s_4: origin xyz=0.6 -0.3 0.0 rpy=0 0 0 -> xyz=0.4 0 0.025 rpy=0 0 0
- joint joint_world_s_0: origin xyz=0.6 -0.15 0.5 rpy=0 0 0 -> xyz=0.5 0 0 rpy=0 0 0; parent ground_link -> world
